File: kicad/data_car/train_distance_car.sch (KiCad schematic (older format))
At the start: 24 parts, among them J1 Encoder Header, J2 Button Header, J3 IFI9431 Header, J4 Button Header, J5 Adafruit 500C Header, U1 Teensy3.2, U2 MB85RS16

Commit message: Update to version 1.2 PCB - fixed parts profiles.  Changes to be committed: 	deleted:    kicad/data_car/sym-lib-table 	deleted:    kicad/data_car/train_distance_car-cache.lib 	deleted:    kicad/data_car/train_distance_car.bak 	deleted:    kicad/data_car/train_distance_car.dsn 	modified:   kicad/data_car/train_distance_car.kicad_pcb 	deleted:    kicad/data_car/train_distance_car.kicad_pcb-bak 	deleted:    kicad/data_car/train_distance_car.net 	deleted:    kicad/data_car/train_distance_car.pro 	deleted:    kicad/data_car/train_distance_car.rules 	modified:   kicad/data_car/train_distance_car.sch 	deleted:    kicad/data_car/train_distance_car.ses 	deleted:    kicad/data_car/train_distance_car_v1.kicad_pcb
Parts:
- added R5, R7: 10k, Resistor_SMD:R_1206_3216Metric, symbol Device:R
- F1: footprint Fuse:Fuse_2920_7451Metric -> Fuse:Fuse_1812_4532Metric_Pad1.30x3.40mm_HandSolder
- U2: footprint Package_SO:SOP-8_6.62x9.15mm_P2.54mm -> Package_SO:SSOP-8_3.9x5.05mm_P1.27mm
- renumbered J3 to J1, J1 to J2, J2 to J3, R5 to R6, R6 to R8, R7 to R9
Connections:
- net +3V3: now also R5.1, R7.1
- net ~FRCS: now also R5.2
- net ~LOBAT: now also U1.25 (18_A4_SDA0_Touch)
- net at U2.3 (~WP): now also U2.7 (~HOLD), R7.2
- net CS renamed ~CS
- net TCS renamed ~TCS
Changed lines of the file:
@@
 Sheet 1 1
 Title "A Carrier Board for Teensy 3.2 and ILI9341 Touch Screet"
-Date "2019-02-22"
-Rev "1.1"
-Comp "Timberlake Hobbies"
-Comment1 ""
-Comment2 "This revision adding in Audio and FRAM for persistent memory"
+Date "2019-03-17"
+Rev "1.2"
+Comp "Designed by:  Eric Timberlake"
+Comment1 "v1.2 fix u1 and f1 pck - add WP and HD pullups"
+Comment2 "v1.0 add beeper and fram for SN and persistent data"
 Comment3 "with a Teensy 3.2 and a few peripherals to make it all more fun..."
 Comment4 "This is a small \"mother board\" to tie together a cheap ILI9431 based touch screen"
@@
 F 0 "U2" H 8500 3328 50  0000 C CNN
 F 1 "MB85RS16" H 8500 3237 50  0000 C CNN
-F 2 "Package_SO:SOP-8_6.62x9.15mm_P2.54mm" H 8150 2800 50  0001 C CNN
+F 2 "Package_SO:SSOP-8_3.9x5.05mm_P1.27mm" H 8150 2800 50  0001 C CNN
 F 3 "http://www.fujitsu.com/downloads/MICRO/fsa/pdf/products/memory/fram/MB85RS16-DS501-00014-6v0-E.pdf" H 8150 2800 50  0001 C CNN
 	1    8500 2850
@@
 MOSI
 Text GLabel 2300 2900 0    50   Input ~ 0
-TCS
+~TCS
 Text GLabel 2300 3000 0    50   Input ~ 0
 SCK
@@
 DnC
 Text GLabel 2300 3700 0    50   Input ~ 0
-CS
+~CS
 Text GLabel 4300 2900 0    50   Input ~ 0
 TIRQ
@@
 MISO
 Text GLabel 4300 3700 0    50   Output ~ 0
-CS
+~CS
 Text GLabel 4300 3600 0    50   Output ~ 0
 DnC
 Text GLabel 4300 3500 0    50   Output ~ 0
-TCS
+~TCS
 Text GLabel 4300 4500 0    50   Output ~ 0
 SCK
@@
 $EndComp
 $Comp
-L power:+3.3V #PWR015
+L power:+3.3V #PWR018
 U 1 1 5C70A5FD
 P 6800 4850
-F 0 "#PWR015" H 6800 4700 50  0001 C CNN
+F 0 "#PWR018" H 6800 4700 50  0001 C CNN
 F 1 "+3.3V" H 6815 5023 50  0000 C CNN
 F 2 "" H 6800 4850 50  0001 C CNN
@@
 $EndComp
 $Comp
-L power:+3.3V #PWR020
+L power:+3.3V #PWR024
 U 1 1 5C70A62F
 P 8500 2300
-F 0 "#PWR020" H 8500 2150 50  0001 C CNN
+F 0 "#PWR024" H 8500 2150 50  0001 C CNN
 F 1 "+3.3V" H 8515 2473 50  0000 C CNN
 F 2 "" H 8500 2300 50  0001 C CNN
@@
 $EndComp
 Wire Wire Line
-	1500 2750 1500 2850
-Wire Wire Line
 	1500 3150 1500 3200
 Wire Wire Line
@@
 $EndComp
 Text GLabel 2650 5000 3    50   Input ~ 0
-TCS
+~TCS
 Text GLabel 3000 5000 3    50   Input ~ 0
-CS
+~CS
 Wire Wire Line
 	2650 4800 2650 5000
@@
 F 0 "F1" V 1645 3900 50  0000 C CNN
 F 1 "450mA Polyfuse" V 1736 3900 50  0000 C CNN
-F 2 "Fuse:Fuse_2920_7451Metric" H 1900 3700 50  0001 L CNN
+F 2 "Fuse:Fuse_1812_4532Metric_Pad1.30x3.40mm_HandSolder" H 1900 3700 50  0001 L CNN
 F 3 "~" H 1850 3900 50  0001 C CNN
 	1    1850 3900
@@
 $EndComp
 $Comp
-L power:+3.3V #PWR016
+L power:+3.3V #PWR019
 U 1 1 5C719D1F
 P 6950 4700
-F 0 "#PWR016" H 6950 4550 50  0001 C CNN
+F 0 "#PWR019" H 6950 4550 50  0001 C CNN
 F 1 "+3.3V" H 6965 4873 50  0000 C CNN
 F 2 "" H 6950 4700 50  0001 C CNN
@@
 $EndComp
 $Comp
-L power:+5V #PWR017
+L power:+5V #PWR021
 U 1 1 5C71BA87
 P 8100 3700
-F 0 "#PWR017" H 8100 3550 50  0001 C CNN
+F 0 "#PWR021" H 8100 3550 50  0001 C CNN
 F 1 "+5V" H 8115 3873 50  0000 C CNN
 F 2 "" H 8100 3700 50  0001 C CNN
@@
 	8100 3750 8350 3750
 $Comp
-L power:GND #PWR018
+L power:GND #PWR022
 U 1 1 5C71E698
 P 8100 4600
-F 0 "#PWR018" H 8100 4350 50  0001 C CNN
+F 0 "#PWR022" H 8100 4350 50  0001 C CNN
 F 1 "GND" H 8105 4427 50  0000 C CNN
 F 2 "" H 8100 4600 50  0001 C CNN
@@
 	8050 4250 8350 4250
 $Comp
-L Device:R R6
+L Device:R R8
 U 1 1 5C724B75
 P 8700 4950
-F 0 "R6" H 8770 4996 50  0000 L CNN
+F 0 "R8" H 8770 4996 50  0000 L CNN
 F 1 "100k" H 8770 4905 50  0000 L CNN
 F 2 "Resistor_SMD:R_1206_3216Metric" V 8630 4950 50  0001 C CNN
@@
 $EndComp
 $Comp
-L Device:R R7
+L Device:R R9
 U 1 1 5C724C0D
 P 8700 5450
-F 0 "R7" H 8770 5496 50  0000 L CNN
+F 0 "R9" H 8770 5496 50  0000 L CNN
 F 1 "100k" H 8770 5405 50  0000 L CNN
 F 2 "Resistor_SMD:R_1206_3216Metric" V 8630 5450 50  0001 C CNN
@@
 VBAT.5
 $Comp
-L power:GND #PWR022
+L power:GND #PWR026
 U 1 1 5C725F53
 P 8700 5800
-F 0 "#PWR022" H 8700 5550 50  0001 C CNN
+F 0 "#PWR026" H 8700 5550 50  0001 C CNN
 F 1 "GND" H 8705 5627 50  0000 C CNN
 F 2 "" H 8700 5800 50  0001 C CNN
@@
 $EndComp
 $Comp
-L power:GND #PWR019
+L power:GND #PWR023
 U 1 1 5C729943
 P 8350 5800
-F 0 "#PWR019" H 8350 5550 50  0001 C CNN
+F 0 "#PWR023" H 8350 5550 50  0001 C CNN
 F 1 "GND" H 8355 5627 50  0000 C CNN
 F 2 "" H 8350 5800 50  0001 C CNN
@@
 	4300 4600 4500 4600
 $Comp
-L Connector:Conn_01x14_Male J3
+L Connector:Conn_01x14_Male J1
 U 1 1 5C72F38F
 P 2650 3200
-F 0 "J3" H 2622 3173 50  0000 R CNN
+F 0 "J1" H 2622 3173 50  0000 R CNN
 F 1 "IFI9431 Header" H 2622 3082 50  0000 R CNN
 F 2 "Connector_PinSocket_2.54mm:PinSocket_1x14_P2.54mm_Vertical" H 2650 3200 50  0001 C CNN
@@
 $EndComp
 $Comp
-L Connector:Conn_01x05_Male J1
+L Connector:Conn_01x05_Male J2
 U 1 1 5C72F7E3
 P 1650 4900
-F 0 "J1" H 1622 4923 50  0000 R CNN
+F 0 "J2" H 1622 4923 50  0000 R CNN
 F 1 "Encoder Header" H 1622 4832 50  0000 R CNN
 F 2 "Connector_PinHeader_2.54mm:PinHeader_1x05_P2.54mm_Vertical" H 1650 4900 50  0001 C CNN
@@
 $EndComp
 $Comp
-L power:GND #PWR021
+L power:GND #PWR025
 U 1 1 5C72FA0A
 P 8500 3300
-F 0 "#PWR021" H 8500 3050 50  0001 C CNN
+F 0 "#PWR025" H 8500 3050 50  0001 C CNN
 F 1 "GND" H 8505 3127 50  0000 C CNN
 F 2 "" H 8500 3300 50  0001 C CNN
@@
 	8500 3150 8500 3300
 $Comp
-L power:+5V #PWR014
+L power:+5V #PWR017
 U 1 1 5C731040
 P 6700 4600
-F 0 "#PWR014" H 6700 4450 50  0001 C CNN
+F 0 "#PWR017" H 6700 4450 50  0001 C CNN
 F 1 "+5V" H 6715 4773 50  0000 C CNN
 F 2 "" H 6700 4600 50  0001 C CNN
@@
 	6800 4900 6800 4850
 $Comp
-L power:GND #PWR013
+L power:GND #PWR016
 U 1 1 5C737049
 P 6550 5450
-F 0 "#PWR013" H 6550 5200 50  0001 C CNN
+F 0 "#PWR016" H 6550 5200 50  0001 C CNN
 F 1 "GND" H 6555 5277 50  0000 C CNN
 F 2 "" H 6550 5450 50  0001 C CNN
@@
 $EndComp
 $Comp
-L Device:R R5
+L Device:R R6
 U 1 1 5C7389D4
 P 3450 6050
-F 0 "R5" H 3520 6096 50  0000 L CNN
+F 0 "R6" H 3520 6096 50  0000 L CNN
 F 1 "10k" H 3520 6005 50  0000 L CNN
 F 2 "Resistor_SMD:R_1206_3216Metric" V 3380 6050 50  0001 C CNN
@@
 $EndComp
 $Comp
-L power:GND #PWR012
+L power:GND #PWR013
 U 1 1 5C738A5E
 P 3450 6500
-F 0 "#PWR012" H 3450 6250 50  0001 C CNN
+F 0 "#PWR013" H 3450 6250 50  0001 C CNN
 F 1 "GND" H 3455 6327 50  0000 C CNN
 F 2 "" H 3450 6500 50  0001 C CNN
@@
 ~BUTTON2
 $Comp
-L power:+3.3V #PWR011
+L power:+3.3V #PWR012
 U 1 1 5C738B06
 P 3450 5800
-F 0 "#PWR011" H 3450 5650 50  0001 C CNN
+F 0 "#PWR012" H 3450 5650 50  0001 C CNN
 F 1 "+3.3V" H 3465 5973 50  0000 C CNN
 F 2 "" H 3450 5800 50  0001 C CNN
@@
 	3450 6400 3450 6500
 $Comp
-L Connector:Conn_01x02_Male J2
+L Connector:Conn_01x02_Male J3
 U 1 1 5C741892
 P 2200 6300
-F 0 "J2" H 2173 6273 50  0000 R CNN
+F 0 "J3" H 2173 6273 50  0000 R CNN
 F 1 "Button Header" H 2173 6182 50  0000 R CNN
 F 2 "Connector_PinHeader_2.54mm:PinHeader_1x02_P2.54mm_Vertical" H 2200 6300 50  0001 C CNN
@@
 	3900 4900 4500 4900
 $Comp
-L power:GND #PWR0101
+L power:GND #PWR015
 U 1 1 5C7270B0
 P 5700 6150
-F 0 "#PWR0101" H 5700 5900 50  0001 C CNN
+F 0 "#PWR015" H 5700 5900 50  0001 C CNN
 F 1 "GND" H 5705 5977 50  0000 C CNN
 F 2 "" H 5700 6150 50  0001 C CNN
@@
 	4900 5950 5150 5950
 $Comp
-L power:GND #PWR0102
+L power:GND #PWR014
 U 1 1 5C732358
 P 3800 2650
-F 0 "#PWR0102" H 3800 2400 50  0001 C CNN
+F 0 "#PWR014" H 3800 2400 50  0001 C CNN
 F 1 "GND" H 3805 2477 50  0000 C CNN
 F 2 "" H 3800 2650 50  0001 C CNN
@@
 	1    0    0    -1
 $EndComp
+Text GLabel 4200 5000 0    50   Input ~ 0
+~LOBAT
+Wire Wire Line
+	4200 5000 4500 5000
+$Comp
+L Device:R R5
+U 1 1 5C83B8A9
+P 3300 4650
+F 0 "R5" H 3370 4696 50  0000 L CNN
+F 1 "10k" H 3370 4605 50  0000 L CNN
+F 2 "Resistor_SMD:R_1206_3216Metric" V 3230 4650 50  0001 C CNN
+F 3 "~" H 3300 4650 50  0001 C CNN
+	1    3300 4650
+	1    0    0    -1
+$EndComp
+$Comp
+L power:+3.3V #PWR011
+U 1 1 5C83B958
+P 3300 4350
+F 0 "#PWR011" H 3300 4200 50  0001 C CNN
+F 1 "+3.3V" H 3315 4523 50  0000 C CNN
+F 2 "" H 3300 4350 50  0001 C CNN
+F 3 "" H 3300 4350 50  0001 C CNN
+	1    3300 4350
+	1    0    0    -1
+$EndComp
+Text GLabel 3300 4950 3    50   Input ~ 0
+~FRCS
+Wire Wire Line
+	3300 4500 3300 4350
+Wire Wire Line
+	3300 4950 3300 4800
+$Comp
+L Device:R R7
+U 1 1 5C844322
+P 7950 2450
+F 0 "R7" H 8020 2496 50  0000 L CNN
+F 1 "10k" H 8020 2405 50  0000 L CNN
+F 2 "Resistor_SMD:R_1206_3216Metric" V 7880 2450 50  0001 C CNN
+F 3 "~" H 7950 2450 50  0001 C CNN
+	1    7950 2450
+	1    0    0    -1
+$EndComp
+$Comp
+L power:+3.3V #PWR020
+U 1 1 5C8443A0
+P 7950 2150
+F 0 "#PWR020" H 7950 2000 50  0001 C CNN
+F 1 "+3.3V" H 7965 2323 50  0000 C CNN
+F 2 "" H 7950 2150 50  0001 C CNN
+F 3 "" H 7950 2150 50  0001 C CNN
+	1    7950 2150
+	1    0    0    -1
+$EndComp
+Wire Wire Line
+	7950 2150 7950 2300
+Wire Wire Line
+	7950 2600 7950 2750
+Wire Wire Line
+	7950 2850 8100 2850
+Wire Wire Line
+	8100 2750 7950 2750
+Connection ~ 7950 2750
+Wire Wire Line
+	7950 2750 7950 2850
+Wire Wire Line
+	1500 2850 1500 2750
 $EndSCHEMATC
